Commit message: fix: refine leg pose to base

File: landing_gear_description/urdf/landing_gear.urdf.xacro (robot description, xacro)
@@ -62,5 +62,5 @@
     <child link="leg"/>
     <!-- the link 1 rotated  ni x rad-->
-    <origin xyz="0 0 -0.1" rpy="-1.5714 3.1415 0"/>
+    <origin xyz="0 -0.0058 -0.105" rpy="-1.5714 3.1415 0"/>
     <axis xyz="-1 0 0"/>
     <limit effort="100" velocity="1" lower="-1.5714" upper="1.5714"/>
@@ -116,5 +116,5 @@
     <child link="leg_2"/>
     <!-- the link 1 rotated  ni x rad-->
-    <origin xyz="0.082 0 0.037" rpy="-1.5714 1.0475 0"/>
+    <origin xyz="0.0856 -0.0058 0.04" rpy="-1.5714 1.0475 0"/>
     <axis xyz="-1 0 0"/>
     <limit effort="100" velocity="1" lower="-1.5714" upper="1.5714"/>
@@ -170,5 +170,5 @@
     <child link="leg_3"/>
     <!-- the link 1 rotated  ni x rad-->
-    <origin xyz="-0.082 0 0.037" rpy="-1.5714 -1.0475 0"/>
+    <origin xyz="-0.083 -0.0058 0.042" rpy="-1.5714 -1.0475 0"/>
     <axis xyz="-1 0 0"/>
     <limit effort="100" velocity="1" lower="-1.5714" upper="1.5714"/>

File: landing_gear_description/urdf/tes.urdf.xacro (robot description, xacro)
@@ -36,4 +36,32 @@
         </inertial>
 </link>
+<!-- leg 2 -->
+<link name="leg_2">
+    <visual>
+        <origin rpy="0 0 0" xyz="0 -0.136 -0.017" />
+        <geometry>
+            <mesh filename="package://landing_gear_description/meshes/link1.stl" scale="0.001 0.001 0.001"/>
+        </geometry>
+    </visual>
+    <collision>
+        <origin rpy="0 0 0" xyz="0 -0.136 -0.017" />
+        <geometry>
+            <mesh filename="package://landing_gear_description/meshes/link1.stl" scale="0.001 0.001 0.001"/>
+        </geometry>
+    </collision>
+    <inertial>
+        <origin rpy="0 0 0" xyz="0 0 0" />
+        <mass value="0.1"/>
+        <inertia ixx="0.001" ixy="0.0" ixz="0.0" iyy="0.001" iyz="0.0" izz="0.001"/>
+    </inertial>
+</link>
+<joint name="base_leg_2_joint" type="revolute">
+    <parent link="base"/>
+    <child link="leg_2"/>
+    <!-- the link 1 rotated  ni x rad-->
+    <origin xyz="-0.0856 -0.0058 0.04" rpy="-1.5714 -1.0475 0"/>
+    <axis xyz="-1 0 0"/>
+    <limit effort="100" velocity="1" lower="-1.5714" upper="1.5714"/>
+</joint>
 <gazebo reference="base" >
     <material> Gazebo/Blue </material>

Commit message: add color and IMU sensor

File: landing_gear_description/urdf/landing_gear.urdf.xacro (robot description, xacro)
@@ -200,7 +200,28 @@
     <limit effort="1000" velocity="1" lower="-1.5714" upper="1.5714"/>
 </joint>
+<!-- gazebo related [colors] -->
 <gazebo reference="base_link" >
-    <material> Gazebo/Blue </material>
-    <kinematic> true </kinematic>
+    <kinematic> false </kinematic>
+</gazebo>
+<gazebo reference="base" >
+    <material> Gazebo/blue </material>
+</gazebo>
+<gazebo reference="leg" >
+    <material> Gazebo/White </material>
+</gazebo>
+<gazebo reference="leg_2" >
+    <material> Gazebo/White </material>
+</gazebo>
+<gazebo reference="leg_3" >
+    <material> Gazebo/White </material>
+</gazebo>
+<gazebo reference="link2_leg" >
+    <material> Gazebo/Yellow </material>
+</gazebo>
+<gazebo reference="link2_leg_2" >
+    <material> Gazebo/Yellow </material>
+</gazebo>
+<gazebo reference="link2_leg_3" >
+    <material> Gazebo/Yellow </material>
 </gazebo>
 <!-- motor controller -->
@@ -229,4 +250,5 @@
     </joint>
 </transmission>
+<!-- leg 2 controller -->
 <transmission name="leg_2_transmission">
     <type>transmission_interfacec/SimpleTransmission</type>
@@ -265,3 +287,38 @@
     </joint>
 </transmission>
+<!-- IMU  -->
+<joint name="imu_joint" type="fixed">
+    <parent link="base_link"/>
+    <child link="imu_link"/>
+    <origin xyz="0.0 0 0" rpy="0 0 0"/>
+  </joint>
+<link name="imu_link"/>
+<!-- gazebo IMU -->
+ <gazebo reference="imu_link">
+    <sensor type="imu" name="imu">
+      <always_on>true</always_on>
+      <visualize>true</visualize>
+    </sensor>
+    <material>Gazebo/Grey</material>
+</gazebo>
+ <gazebo reference="imu_link">
+    <gravity>true</gravity>
+    <sensor name="imu_sensor" type="imu">
+      <always_on>true</always_on>
+      <update_rate>100</update_rate>
+      <visualize>true</visualize>
+      <topic>__default_topic__</topic>
+      <plugin filename="libgazebo_ros_imu_sensor.so" name="imu_plugin">
+        <topicName>imu</topicName>
+        <bodyName>imu_link</bodyName>
+        <updateRateHZ>10.0</updateRateHZ>
+        <gaussianNoise>0.0</gaussianNoise>
+        <xyzOffset>0 0 0</xyzOffset>
+        <rpyOffset>0 0 0</rpyOffset>
+        <frameName>imu_link</frameName>
+        <initialOrientationAsReference>false</initialOrientationAsReference>
+      </plugin>
+      <pose>0 0 0 0 0 0</pose>
+    </sensor>
+</gazebo>
 </robot>

Commit message: change color

File: landing_gear_description/urdf/landing_gear.urdf.xacro (robot description, xacro)
@@ -205,5 +205,5 @@
 </gazebo>
 <gazebo reference="base" >
-    <material> Gazebo/blue </material>
+    <material> Gazebo/Gray </material>
 </gazebo>
 <gazebo reference="leg" >
@@ -211,11 +211,11 @@
 </gazebo>
 <gazebo reference="leg_2" >
+    <material> Gazebo/Yellow </material>
+</gazebo>
+<gazebo reference="leg_3" >
+    <material> Gazebo/Blue </material>
+</gazebo>
+<gazebo reference="link2_leg" >
     <material> Gazebo/White </material>
-</gazebo>
-<gazebo reference="leg_3" >
-    <material> Gazebo/White </material>
-</gazebo>
-<gazebo reference="link2_leg" >
-    <material> Gazebo/Yellow </material>
 </gazebo>
 <gazebo reference="link2_leg_2" >
@@ -223,5 +223,5 @@
 </gazebo>
 <gazebo reference="link2_leg_3" >
-    <material> Gazebo/Yellow </material>
+    <material> Gazebo/Blue </material>
 </gazebo>
 <!-- motor controller -->

Commit message: change leg joint naming

File: landing_gear_description/urdf/landing_gear.urdf.xacro (robot description, xacro)
@@ -58,5 +58,5 @@
     </inertial>
 </link>
-<joint name="base_leg_joint" type="revolute">
+<joint name="base_leg_1_joint" type="revolute">
     <parent link="base"/>
     <child link="leg"/>
@@ -85,10 +85,10 @@
     </inertial>
 </link>
-<joint name="base_link2_leg_joint" type="revolute">
+<joint name="base_link2_leg_1_joint" type="revolute">
     <parent link="leg"/>
     <child link="link2_leg"/>
     <origin xyz="0 -0.12 0" rpy="-1.5714 0 0"/>
     <axis xyz="1 0 0"/>
-    <limit effort="1000" velocity="1" lower="-3.1415" upper="3.1415"/>
+    <limit effort="100" velocity="1" lower="-3.1415" upper="3.1415"/>
 </joint>
 <!-- leg 2 -->
@@ -144,5 +144,5 @@
     <origin xyz="0 -0.12 0" rpy="-1.5714 0 0"/>
     <axis xyz="1 0 0"/>
-    <limit effort="1000" velocity="1" lower="-1.5714" upper="1.5714"/>
+    <limit effort="100" velocity="1" lower="-1.5714" upper="1.5714"/>
 </joint>
 <!-- leg 3 -->
@@ -198,9 +198,9 @@
     <origin xyz="0 -0.12 0" rpy="-1.5714 0 0"/>
     <axis xyz="1 0 0"/>
-    <limit effort="1000" velocity="1" lower="-1.5714" upper="1.5714"/>
+    <limit effort="100" velocity="1" lower="-1.5714" upper="1.5714"/>
 </joint>
 <!-- gazebo related [colors] -->
 <gazebo reference="base_link" >
-    <kinematic> false </kinematic>
+    <kinematic> true </kinematic>
 </gazebo>
 <gazebo reference="base" >
@@ -237,5 +237,5 @@
         <mechanicalReduction>1</mechanicalReduction>
     </actuator>
-    <joint name="base_leg_joint">
+    <joint name="base_leg_1_joint">
         <hardwareInterface>hardware_interface/EffortJointInterface</hardwareInterface>
     </joint>
@@ -246,5 +246,5 @@
         <mechanicalReduction>1</mechanicalReduction>
     </actuator>
-    <joint name="base_link2_leg_joint">
+    <joint name="base_link2_leg_1_joint">
         <hardwareInterface>hardware_interface/EffortJointInterface</hardwareInterface>
     </joint>

Commit message: add: Lidar on each leg working

File: landing_gear_description/urdf/landing_gear.urdf.xacro (robot description, xacro)
@@ -322,3 +322,145 @@
     </sensor>
 </gazebo>
+<!-- lidar sensor -->
+<!-- lidar leg1 -->
+<link name="base_scan">
+    <origin rpy="0 0 0" xyz="0 0 0" />
+    <inertial>
+        <origin xyz="0.0 0.0 0.0" rpy="0.0 0.0 0.0"/>
+        <mass value="0.0001"/>
+        <inertia ixx="1" ixy="0.0" ixz="0" iyy="1" iyz="0.0" izz="1"/>
+    </inertial>
+</link>
+<joint name="scan_joint" type="fixed">
+    <parent link="link2_leg"/>
+    <child link="base_scan"/>
+    <origin xyz="0 0.05 0" rpy="0 0 1.57"/>
+    <axis xyz="1 0 0"/>
+</joint>
+<gazebo reference="base_scan">
+    <gravity>true</gravity>
+    <sensor type="ray" name="laser_scan">
+        <pose>0 0 0 0 0 0</pose>
+        <visualize>true</visualize>
+        <always_on>true</always_on>
+        <update_rate>5</update_rate>
+        <ray>
+            <scan>
+            <horizontal>
+              <samples>1</samples>
+              <resolution>1</resolution>
+            </horizontal>
+            </scan>
+            <range>
+                <min>0.01</min>
+                <max>2</max>
+                <resolution>0.015</resolution>
+            </range>
+            <noise>
+                <type>gaussian</type>
+                <mean>0.0</mean>
+                <stddev>0.0</stddev>
+            </noise>
+        </ray>
+        <plugin name="gazebo_ros_scan_controller" filename="libgazebo_ros_laser.so">
+            <robotNamespace>lg</robotNamespace>
+            <topicName>lidar1</topicName>
+            <frameName>base_scan</frameName>
+        </plugin>
+    </sensor>
+</gazebo>
+<!-- lidar leg2 -->
+<link name="base_scan2">
+    <origin rpy="0 0 0" xyz="0 0 0" />
+    <inertial>
+        <origin xyz="0.0 0.0 0.0" rpy="0.0 0.0 0.0"/>
+        <mass value="0.0001"/>
+        <inertia ixx="1" ixy="0.0" ixz="0" iyy="1" iyz="0.0" izz="1"/>
+    </inertial>
+</link>
+<joint name="scan2_joint" type="fixed">
+    <parent link="link2_leg_2"/>
+    <child link="base_scan2"/>
+    <origin xyz="0 0.05 0" rpy="0 0 1.57"/>
+    <axis xyz="1 0 0"/>
+</joint>
+<gazebo reference="base_scan2">
+    <gravity>true</gravity>
+    <sensor type="ray" name="laser_scan2">
+        <pose>0 0 0 0 0 0</pose>
+        <visualize>true</visualize>
+        <always_on>true</always_on>
+        <update_rate>5</update_rate>
+        <ray>
+            <scan>
+            <horizontal>
+              <samples>1</samples>
+              <resolution>1</resolution>
+            </horizontal>
+            </scan>
+            <range>
+                <min>0.01</min>
+                <max>2</max>
+                <resolution>0.015</resolution>
+            </range>
+            <noise>
+                <type>gaussian</type>
+                <mean>0.0</mean>
+                <stddev>0.0</stddev>
+            </noise>
+        </ray>
+        <plugin name="gazebo_ros_scan_controller" filename="libgazebo_ros_laser.so">
+            <robotNamespace>lg</robotNamespace>
+            <topicName>lidar2</topicName>
+            <frameName>base_scan2</frameName>
+        </plugin>
+    </sensor>
+</gazebo>
+<!-- lidar leg3 -->
+<link name="base_scan3">
+    <origin rpy="0 0 0" xyz="0 0 0" />
+    <inertial>
+        <origin xyz="0.0 0.0 0.0" rpy="0.0 0.0 0.0"/>
+        <mass value="0.0001"/>
+        <inertia ixx="1" ixy="0.0" ixz="0" iyy="1" iyz="0.0" izz="1"/>
+    </inertial>
+</link>
+<joint name="scan3_joint" type="fixed">
+    <parent link="link2_leg_3"/>
+    <child link="base_scan3"/>
+    <origin xyz="0 0.05 0" rpy="0 0 1.57"/>
+    <axis xyz="1 0 0"/>
+</joint>
+<gazebo reference="base_scan3">
+    <gravity>true</gravity>
+    <sensor type="ray" name="laser_scan3">
+        <pose>0 0 0 0 0 0</pose>
+        <visualize>true</visualize>
+        <always_on>true</always_on>
+        <update_rate>5</update_rate>
+        <ray>
+            <scan>
+            <horizontal>
+              <samples>1</samples>
+              <resolution>1</resolution>
+            </horizontal>
+            </scan>
+            <range>
+                <min>0.01</min>
+                <max>2</max>
+                <resolution>0.015</resolution>
+            </range>
+            <noise>
+                <type>gaussian</type>
+                <mean>0.0</mean>
+                <stddev>0.0</stddev>
+            </noise>
+        </ray>
+        <plugin name="gazebo_ros_scan_controller" filename="libgazebo_ros_laser.so">
+            <robotNamespace>lg</robotNamespace>
+            <topicName>lidar3</topicName>
+            <frameName>base_scan3</frameName>
+        </plugin>
+    </sensor>
+</gazebo>
 </robot>
