Commit message: refactor: cleanup urdf, split urdf definition and use macro for legs

File: landing_gear_description/urdf/landing_gear.urdf.xacro (robot description, xacro)
@@ -1,8 +1,6 @@
 <?xml version="1.0" ?>
 <robot name="landing_gear" xmlns:xacro="http://ros.org/wiki/xacro">
-    <!-- <xacro:property name="link1_length" value="0.2"/>
-    <xacro:property name="link1_radius" value="0.02"/> -->
-<xacro:property name="base_r" value="0.2"/>
-<xacro:property name="base_d" value="0.002"/>
+<xacro:include filename="$(find landing_gear_description)/urdf/landing_gear.gazebo.xacro"/>
+<xacro:include filename="$(find landing_gear_description)/urdf/leg.urdf.xacro"/>
 <!-- Base Link -->
 <link name="base_link">
@@ -38,253 +36,7 @@
         </inertial>
 </link>
-<!-- leg 1 -->
-<link name="leg">
-    <visual>
-        <origin rpy="0 0 0" xyz="0 -0.136 -0.017" />
-        <geometry>
-            <mesh filename="package://landing_gear_description/meshes/link1.stl" scale="0.001 0.001 0.001"/>
-        </geometry>
-    </visual>
-    <collision>
-        <origin rpy="0 0 0" xyz="0 -0.136 -0.017" />
-        <geometry>
-            <mesh filename="package://landing_gear_description/meshes/link1.stl" scale="0.001 0.001 0.001"/>
-        </geometry>
-    </collision>
-    <inertial>
-        <origin rpy="0 0 0" xyz="0 0 0" />
-        <mass value="0.1"/>
-        <inertia ixx="0.001" ixy="0.0" ixz="0.0" iyy="0.001" iyz="0.0" izz="0.001"/>
-    </inertial>
-</link>
-<joint name="base_leg_1_joint" type="revolute">
-    <parent link="base"/>
-    <child link="leg"/>
-    <!-- the link 1 rotated  ni x rad-->
-    <origin xyz="0 -0.0058 -0.105" rpy="-1.5714 3.1415 0"/>
-    <axis xyz="-1 0 0"/>
-    <limit effort="100" velocity="1" lower="-1.5714" upper="1.5714"/>
-</joint>
-<link name="link2_leg">
-    <visual>
-        <origin rpy="0 0 0" xyz="0.01 0.0125 -0.0125" />
-        <geometry>
-            <mesh filename="package://landing_gear_description/meshes/link2.stl" scale="0.001 0.001 0.001"/>
-        </geometry>
-    </visual>
-    <collision>
-        <origin rpy="0 0 0" xyz="0.01 0.0125 -0.0125" />
-        <geometry>
-            <mesh filename="package://landing_gear_description/meshes/link2.stl" scale="0.001 0.001 0.001"/>
-        </geometry>
-    </collision>
-    <inertial>
-        <origin rpy="0 0 0" xyz="0 0 0" />
-        <mass value="0.1"/>
-        <inertia ixx="0.001" ixy="0.0" ixz="0.0" iyy="0.001" iyz="0.0" izz="0.001"/>
-    </inertial>
-</link>
-<joint name="base_link2_leg_1_joint" type="revolute">
-    <parent link="leg"/>
-    <child link="link2_leg"/>
-    <origin xyz="0 -0.12 0" rpy="-1.5714 0 0"/>
-    <axis xyz="1 0 0"/>
-    <limit effort="100" velocity="1" lower="-3.1415" upper="3.1415"/>
-</joint>
-<!-- leg 2 -->
-<link name="leg_2">
-    <visual>
-        <origin rpy="0 0 0" xyz="0 -0.136 -0.017" />
-        <geometry>
-            <mesh filename="package://landing_gear_description/meshes/link1.stl" scale="0.001 0.001 0.001"/>
-        </geometry>
-    </visual>
-    <collision>
-        <origin rpy="0 0 0" xyz="0 -0.136 -0.017" />
-        <geometry>
-            <mesh filename="package://landing_gear_description/meshes/link1.stl" scale="0.001 0.001 0.001"/>
-        </geometry>
-    </collision>
-    <inertial>
-        <origin rpy="0 0 0" xyz="0 0 0" />
-        <mass value="0.1"/>
-        <inertia ixx="0.001" ixy="0.0" ixz="0.0" iyy="0.001" iyz="0.0" izz="0.001"/>
-    </inertial>
-</link>
-<joint name="base_leg_2_joint" type="revolute">
-    <parent link="base"/>
-    <child link="leg_2"/>
-    <!-- the link 1 rotated  ni x rad-->
-    <origin xyz="0.0856 -0.0058 0.04" rpy="-1.5714 1.0475 0"/>
-    <axis xyz="-1 0 0"/>
-    <limit effort="100" velocity="1" lower="-1.5714" upper="1.5714"/>
-</joint>
-<link name="link2_leg_2">
-    <visual>
-        <origin rpy="0 0 0" xyz="0.01 0.0125 -0.0125" />
-        <geometry>
-            <mesh filename="package://landing_gear_description/meshes/link2.stl" scale="0.001 0.001 0.001"/>
-        </geometry>
-    </visual>
-    <collision>
-        <origin rpy="0 0 0" xyz="0.01 0.0125 -0.0125" />
-        <geometry>
-            <mesh filename="package://landing_gear_description/meshes/link2.stl" scale="0.001 0.001 0.001"/>
-        </geometry>
-    </collision>
-    <inertial>
-        <origin rpy="0 0 0" xyz="0 0 0" />
-        <mass value="0.1"/>
-        <inertia ixx="0.001" ixy="0.0" ixz="0.0" iyy="0.001" iyz="0.0" izz="0.001"/>
-    </inertial>
-</link>
-<joint name="base_link2_leg_2_joint" type="revolute">
-    <parent link="leg_2"/>
-    <child link="link2_leg_2"/>
-    <origin xyz="0 -0.12 0" rpy="-1.5714 0 0"/>
-    <axis xyz="1 0 0"/>
-    <limit effort="100" velocity="1" lower="-1.5714" upper="1.5714"/>
-</joint>
-<!-- leg 3 -->
-<link name="leg_3">
-    <visual>
-        <origin rpy="0 0 0" xyz="0 -0.136 -0.017" />
-        <geometry>
-            <mesh filename="package://landing_gear_description/meshes/link1.stl" scale="0.001 0.001 0.001"/>
-        </geometry>
-    </visual>
-    <collision>
-        <origin rpy="0 0 0" xyz="0 -0.136 -0.017" />
-        <geometry>
-            <mesh filename="package://landing_gear_description/meshes/link1.stl" scale="0.001 0.001 0.001"/>
-        </geometry>
-    </collision>
-    <inertial>
-        <origin rpy="0 0 0" xyz="0 0 0" />
-        <mass value="0.1"/>
-        <inertia ixx="0.001" ixy="0.0" ixz="0.0" iyy="0.001" iyz="0.0" izz="0.001"/>
-    </inertial>
-</link>
-<joint name="base_leg_3_joint" type="revolute">
-    <parent link="base"/>
-    <child link="leg_3"/>
-    <!-- the link 1 rotated  ni x rad-->
-    <origin xyz="-0.083 -0.0058 0.042" rpy="-1.5714 -1.0475 0"/>
-    <axis xyz="-1 0 0"/>
-    <limit effort="100" velocity="1" lower="-1.5714" upper="1.5714"/>
-</joint>
-<link name="link2_leg_3">
-    <visual>
-        <origin rpy="0 0 0" xyz="0.01 0.0125 -0.0125" />
-        <geometry>
-            <mesh filename="package://landing_gear_description/meshes/link2.stl" scale="0.001 0.001 0.001"/>
-        </geometry>
-    </visual>
-    <collision>
-        <origin rpy="0 0 0" xyz="0.01 0.0125 -0.0125" />
-        <geometry>
-            <mesh filename="package://landing_gear_description/meshes/link2.stl" scale="0.001 0.001 0.001"/>
-        </geometry>
-    </collision>
-    <inertial>
-        <origin rpy="0 0 0" xyz="0 0 0" />
-        <mass value="0.1"/>
-        <inertia ixx="0.001" ixy="0.0" ixz="0.0" iyy="0.001" iyz="0.0" izz="0.001"/>
-    </inertial>
-</link>
-<joint name="base_link2_leg_3_joint" type="revolute">
-    <parent link="leg_3"/>
-    <child link="link2_leg_3"/>
-    <origin xyz="0 -0.12 0" rpy="-1.5714 0 0"/>
-    <axis xyz="1 0 0"/>
-    <limit effort="100" velocity="1" lower="-1.5714" upper="1.5714"/>
-</joint>
-<!-- gazebo related [colors] -->
-<gazebo reference="base_link" >
-    <kinematic> true </kinematic>
-</gazebo>
-<gazebo reference="base" >
-    <material> Gazebo/Gray </material>
-</gazebo>
-<gazebo reference="leg" >
-    <material> Gazebo/White </material>
-</gazebo>
-<gazebo reference="leg_2" >
-    <material> Gazebo/Yellow </material>
-</gazebo>
-<gazebo reference="leg_3" >
-    <material> Gazebo/Blue </material>
-</gazebo>
-<gazebo reference="link2_leg" >
-    <material> Gazebo/White </material>
-</gazebo>
-<gazebo reference="link2_leg_2" >
-    <material> Gazebo/Yellow </material>
-</gazebo>
-<gazebo reference="link2_leg_3" >
-    <material> Gazebo/Blue </material>
-</gazebo>
-<!-- motor controller -->
-<gazebo>
-    <plugin name="gazebo_ros_control" filename="libgazebo_ros_control.so">
-        <robotNamespace>landing_gear</robotNamespace>
-    </plugin>
-</gazebo>
-<!-- leg 1 controller -->
-<transmission name="leg_transmission">
-    <type>transmission_interfacec/SimpleTransmission</type>
-    <actuator name="motor1">
-        <mechanicalReduction>1</mechanicalReduction>
-    </actuator>
-    <joint name="base_leg_1_joint">
-        <hardwareInterface>hardware_interface/EffortJointInterface</hardwareInterface>
-    </joint>
-</transmission>
-<transmission name="leg_1_2_transmission">
-    <type>transmission_interfacec/SimpleTransmission</type>
-    <actuator name="motor1_2">
-        <mechanicalReduction>1</mechanicalReduction>
-    </actuator>
-    <joint name="base_link2_leg_1_joint">
-        <hardwareInterface>hardware_interface/EffortJointInterface</hardwareInterface>
-    </joint>
-</transmission>
-<!-- leg 2 controller -->
-<transmission name="leg_2_transmission">
-    <type>transmission_interfacec/SimpleTransmission</type>
-    <actuator name="motor2">
-        <mechanicalReduction>1</mechanicalReduction>
-    </actuator>
-    <joint name="base_leg_2_joint">
-        <hardwareInterface>hardware_interface/EffortJointInterface</hardwareInterface>
-    </joint>
-</transmission>
-<transmission name="leg_2_2_transmission">
-    <type>transmission_interfacec/SimpleTransmission</type>
-    <actuator name="motor2_2">
-        <mechanicalReduction>1</mechanicalReduction>
-    </actuator>
-    <joint name="base_link2_leg_2_joint">
-        <hardwareInterface>hardware_interface/EffortJointInterface</hardwareInterface>
-    </joint>
-</transmission>
-<transmission name="leg_3_transmission">
-    <type>transmission_interfacec/SimpleTransmission</type>
-    <actuator name="motor3">
-        <mechanicalReduction>1</mechanicalReduction>
-    </actuator>
-    <joint name="base_leg_3_joint">
-        <hardwareInterface>hardware_interface/EffortJointInterface</hardwareInterface>
-    </joint>
-</transmission>
-<transmission name="leg_3_2_transmission">
-    <type>transmission_interfacec/SimpleTransmission</type>
-    <actuator name="motor3_2">
-        <mechanicalReduction>1</mechanicalReduction>
-    </actuator>
-    <joint name="base_link2_leg_3_joint">
-        <hardwareInterface>hardware_interface/EffortJointInterface</hardwareInterface>
-    </joint>
-</transmission>
+<xacro:leg postfix="1" x="0" y="-0.0058" z="-0.105" R="-1.5714" P="3.1415" Y="0"/>
+<xacro:leg postfix="2" x="0.0856" y="-0.0058" z="0.04" R="-1.5714" P="1.0475" Y="0"/>
+<xacro:leg postfix="3" x="-0.083" y="-0.0058" z="0.04" R="-1.5714" P="-1.0475" Y="0"/>
 <!-- IMU  -->
 <joint name="imu_joint" type="fixed">
@@ -322,145 +74,3 @@
     </sensor>
 </gazebo>
-<!-- lidar sensor -->
-<!-- lidar leg1 -->
-<link name="base_scan">
-    <origin rpy="0 0 0" xyz="0 0 0" />
-    <inertial>
-        <origin xyz="0.0 0.0 0.0" rpy="0.0 0.0 0.0"/>
-        <mass value="0.0001"/>
-        <inertia ixx="1" ixy="0.0" ixz="0" iyy="1" iyz="0.0" izz="1"/>
-    </inertial>
-</link>
-<joint name="scan_joint" type="fixed">
-    <parent link="link2_leg"/>
-    <child link="base_scan"/>
-    <origin xyz="0 0.05 0" rpy="0 0 1.57"/>
-    <axis xyz="1 0 0"/>
-</joint>
-<gazebo reference="base_scan">
-    <gravity>true</gravity>
-    <sensor type="ray" name="laser_scan">
-        <pose>0 0 0 0 0 0</pose>
-        <visualize>true</visualize>
-        <always_on>true</always_on>
-        <update_rate>5</update_rate>
-        <ray>
-            <scan>
-            <horizontal>
-              <samples>1</samples>
-              <resolution>1</resolution>
-            </horizontal>
-            </scan>
-            <range>
-                <min>0.01</min>
-                <max>2</max>
-                <resolution>0.015</resolution>
-            </range>
-            <noise>
-                <type>gaussian</type>
-                <mean>0.0</mean>
-                <stddev>0.0</stddev>
-            </noise>
-        </ray>
-        <plugin name="gazebo_ros_scan_controller" filename="libgazebo_ros_laser.so">
-            <robotNamespace>lg</robotNamespace>
-            <topicName>lidar1</topicName>
-            <frameName>base_scan</frameName>
-        </plugin>
-    </sensor>
-</gazebo>
-<!-- lidar leg2 -->
-<link name="base_scan2">
-    <origin rpy="0 0 0" xyz="0 0 0" />
-    <inertial>
-        <origin xyz="0.0 0.0 0.0" rpy="0.0 0.0 0.0"/>
-        <mass value="0.0001"/>
-        <inertia ixx="1" ixy="0.0" ixz="0" iyy="1" iyz="0.0" izz="1"/>
-    </inertial>
-</link>
-<joint name="scan2_joint" type="fixed">
-    <parent link="link2_leg_2"/>
-    <child link="base_scan2"/>
-    <origin xyz="0 0.05 0" rpy="0 0 1.57"/>
-    <axis xyz="1 0 0"/>
-</joint>
-<gazebo reference="base_scan2">
-    <gravity>true</gravity>
-    <sensor type="ray" name="laser_scan2">
-        <pose>0 0 0 0 0 0</pose>
-        <visualize>true</visualize>
-        <always_on>true</always_on>
-        <update_rate>5</update_rate>
-        <ray>
-            <scan>
-            <horizontal>
-              <samples>1</samples>
-              <resolution>1</resolution>
-            </horizontal>
-            </scan>
-            <range>
-                <min>0.01</min>
-                <max>2</max>
-                <resolution>0.015</resolution>
-            </range>
-            <noise>
-                <type>gaussian</type>
-                <mean>0.0</mean>
-                <stddev>0.0</stddev>
-            </noise>
-        </ray>
-        <plugin name="gazebo_ros_scan_controller" filename="libgazebo_ros_laser.so">
-            <robotNamespace>lg</robotNamespace>
-            <topicName>lidar2</topicName>
-            <frameName>base_scan2</frameName>
-        </plugin>
-    </sensor>
-</gazebo>
-<!-- lidar leg3 -->
-<link name="base_scan3">
-    <origin rpy="0 0 0" xyz="0 0 0" />
-    <inertial>
-        <origin xyz="0.0 0.0 0.0" rpy="0.0 0.0 0.0"/>
-        <mass value="0.0001"/>
-        <inertia ixx="1" ixy="0.0" ixz="0" iyy="1" iyz="0.0" izz="1"/>
-    </inertial>
-</link>
-<joint name="scan3_joint" type="fixed">
-    <parent link="link2_leg_3"/>
-    <child link="base_scan3"/>
-    <origin xyz="0 0.05 0" rpy="0 0 1.57"/>
-    <axis xyz="1 0 0"/>
-</joint>
-<gazebo reference="base_scan3">
-    <gravity>true</gravity>
-    <sensor type="ray" name="laser_scan3">
-        <pose>0 0 0 0 0 0</pose>
-        <visualize>true</visualize>
-        <always_on>true</always_on>
-        <update_rate>5</update_rate>
-        <ray>
-            <scan>
-            <horizontal>
-              <samples>1</samples>
-              <resolution>1</resolution>
-            </horizontal>
-            </scan>
-            <range>
-                <min>0.01</min>
-                <max>2</max>
-                <resolution>0.015</resolution>
-            </range>
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